File: ESP32_Shield/ESP32_Shield.kicad_sch (KiCad schematic)
At the start: 25 parts, among them J1 Conn_01x19_Female, J2 Conn_01x19_Female, J3 Conn_01x19_Female, J4 Conn_01x19_Female, J5 Screw_Terminal_01x03, J6 Screw_Terminal_01x03, J7 Screw_Terminal_01x03, K1 FINDER-36.11, K2 FINDER-36.11, K3 FINDER-36.11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

Commit message: PCB: layout completeded
Parts:
- added H1, H2, H3, H4: MountingHole, MountingHole:MountingHole_2.2mm_M2, symbol Mechanical:MountingHole
- D1, D2, D5: footprint Diode_THT:D_DO-41_SOD81_P10.16mm_Horizontal -> Diode_SMD:D_0805_2012Metric
- D3, D4, D6: footprint (none) -> LED_SMD:LED_0805_2012Metric
- J1, J2, J3, J4: footprint Package_DFN_QFN:QFN-48-1EP_7x7mm_P0.5mm_EP5.45x5.45mm_ThermalVias -> Connector_PinHeader_2.54mm:PinHeader_1x19_P2.54mm_Vertical
- J5, J6, J7: footprint (none) -> TerminalBlock:TerminalBlock_Altech_AK300-3_P5.00mm
- Q1, Q2, Q3: footprint Package_TO_SOT_THT:TO-92_Inline -> Package_TO_SOT_SMD:SOT-23
- R1, R2, R5: value 1K -> 330; footprint (none) -> Resistor_SMD:R_0805_2012Metric
- R3, R4, R6: footprint (none) -> Resistor_SMD:R_0805_2012Metric
Connections:
- net 5V is gone; now on net +5V: J2.1 (Pin_1), J4.1 (Pin_1)
- net +5V: now also J4.17 (Pin_17), J4.18 (Pin_18); no longer D1.1 (K), D2.1 (K), D5.1 (K), K1.A1, K2.A1, K3.A1, R1.1, R2.1, R5.1
- net COM: no longer J6.2 (Pin_2), J7.2 (Pin_2), K2.11, K3.11
- net D0: now also R6.1
- net D2: now also R4.1
- net D4: now also R3.1
- net EN: no longer J4.18 (Pin_18)
- net GND: now also J3.15 (Pin_15), J3.16 (Pin_16)
- net NA: no longer J6.1 (Pin_1), J7.1 (Pin_1), K2.14, K3.14
- net NC: no longer J6.3 (Pin_3), J7.3 (Pin_3), K2.12, K3.12
- net RX: no longer J3.15 (Pin_15)
- net TX: no longer J3.16 (Pin_16)
- net VP: no longer J4.17 (Pin_17)
- net 3V3 renamed +3.3V
- net +3.3V: now also D1.1 (K), D2.1 (K), D5.1 (K), K1.A1, K2.A1, K3.A1, R1.1, R2.1, R5.1
- removed net GPIO6: R3.1, R4.1, R6.1
- new net COM2: J6.2 (Pin_2), K2.11
- new net COM3: J7.2 (Pin_2), K3.11
- new net NA2: J6.1 (Pin_1), K2.14
- new net NA3: J7.1 (Pin_1), K3.14
- new net NC2: J6.3 (Pin_3), K2.12
- new net NC3: J7.3 (Pin_3), K3.12
Other:
- moved on the sheet: J2, J4
